Commit message: Add files via upload

File: mycobot_moveit/config/urdf/mycobot_320_m5_custom.urdf (robot description, URDF)
Before this commit: robot firefighter, 7 links, 6 joints
Links:
- link base: geometry collision mesh filename=package://mycobot_moveit/config/urdf/base.stl; visual mesh filename=package://mycobot_moveit/config/urdf/base.stl
- link link1: geometry collision mesh filename=package://mycobot_moveit/config/urdf/link1.stl; visual mesh filename=package://mycobot_moveit/config/urdf/link1.stl
- link link2: geometry collision mesh filename=package://mycobot_moveit/config/urdf/link2.stl; visual mesh filename=package://mycobot_moveit/config/urdf/link2.stl
- link link3: geometry collision mesh filename=package://mycobot_moveit/config/urdf/link3.stl; visual mesh filename=package://mycobot_moveit/config/urdf/link3.stl
- link link4: geometry collision mesh filename=package://mycobot_moveit/config/urdf/link4.stl; visual mesh filename=package://mycobot_moveit/config/urdf/link4.stl
- link link5: geometry collision mesh filename=package://mycobot_moveit/config/urdf/link5.stl; visual mesh filename=package://mycobot_moveit/config/urdf/link5.stl
- link link6: geometry collision mesh filename=package://mycobot_moveit/config/urdf/link6.stl; visual mesh filename=package://mycobot_moveit/config/urdf/link6.stl
Joints:
- joint joint3_to_joint2: origin xyz=0 0 0.0709 rpy=0 0 0 -> xyz=0.0 0.055 0.0709 rpy=0 0 0
- joint joint4_to_joint3: origin xyz=0 0 0.135 rpy=0 0 0 -> xyz=-0.0 -0.01 0.135 rpy=0 0 0
- joint joint6_to_joint5: origin xyz=0 0.088779 0.0461 rpy=0 0 0 -> xyz=0.0 0.04378 0.0461 rpy=0 0 0
- joint joint6output_to_joint6: origin xyz=0 0.0655 0.051 rpy=0 0 0 -> xyz=0.0 0.0455 0.049 rpy=0 0 0
