Commit message: Add files via upload

File: mycobot_with_gripper/config/urdf/mycobot_320_m5_custom.urdf (robot description, URDF)
Before this commit: robot mycobot_320, 19 links, 18 joints
Links:
- removed link camera
- link base: geometry collision mesh filename=package://mycobot_with_gripper/config/urdf/base.obj; visual mesh filename=package://mycobot_with_gripper/config/urdf/base.obj
- link gripper_holder: geometry collision mesh filename=package://mycobot_with_gripper/config/urdf/gripper_holder.o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; visual mesh filename=package://mycobot_with_gripper/config/urdf/gripper_holder.o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
- link gripperlink: geometry collision mesh filename=package://mycobot_with_gripper/config/urdf/gripperlink.obj; visual mesh filename=package://mycobot_with_gripper/config/urdf/gripperlink.obj
- link hand_base_link: geometry collision mesh filename=package://mycobot_with_gripper/config/urdf/hand_base_link.o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; visual mesh filename=package://mycobot_with_gripper/config/urdf/hand_base_link.o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
- link link1: geometry collision mesh filename=package://mycobot_with_gripper/config/urdf/link1.obj; visual mesh filename=package://mycobot_with_gripper/config/urdf/link1.obj
- link link2: geometry collision mesh filename=package://mycobot_with_gripper/config/urdf/link2.obj; visual mesh filename=package://mycobot_with_gripper/config/urdf/link2.obj
- link link3: geometry collision mesh filename=package://mycobot_with_gripper/config/urdf/link3.obj; visual mesh filename=package://mycobot_with_gripper/config/urdf/link3.obj
- link link4: geometry collision mesh filename=package://mycobot_with_gripper/config/urdf/link4.obj; visual mesh filename=package://mycobot_with_gripper/config/urdf/link4.obj
- link link5: geometry collision mesh filename=package://mycobot_with_gripper/config/urdf/link5.obj; visual mesh filename=package://mycobot_with_gripper/config/urdf/link5.obj
- link link6: geometry collision mesh filename=package://mycobot_with_gripper/config/urdf/link6.obj; visual mesh filename=package://mycobot_with_gripper/config/urdf/link6.obj
Joints:
- removed joint camera_joint
- joint gripperlink joint: parent camera -> link6
